File: SafeGuardBuzzer_v1.kicad_sch (KiCad schematic)
At the start: 16 parts, among them J1 SWD_DEBUG_PADS, J2 VBAT_RAW_GND_TEST_PADS, Q1 AO3400A logic-level NMOS, U1 DA14531MOD-00F01002

Commit message: Update Buzzer JLC BOM metadata and corrected CPL origin
Parts:
- BT1, BZ1: JLCPCB_Type (none) -> Extended
- C1: JLCPCB_Type (none) -> Basic; LCSC (none) -> C440198; MPN (none) -> GRM21BR61H106KE43L; Manufacturer Generic -> Murata
- C2: JLCPCB_Type (none) -> Basic; LCSC (none) -> C14663; MPN (none) -> CC0603KRX7R9BB104; Manufacturer Generic -> YAGEO
- C3: JLCPCB_Type (none) -> Extended; LCSC (none) -> C49066; MPN (none) -> CL32A107MQVNNNE; Manufacturer Generic -> Samsung Electro-Mechanics
- D1: JLCPCB_Type (none) -> Basic; LCSC (none) -> C2286; MPN (none) -> KT-0603R; Manufacturer Generic -> KENTO
- D2: JLCPCB_Type (none) -> Extended; LCSC (none) -> C22629; MPN BAT54WS -> BAT54WS L9
- Q1: JLCPCB_Type (none) -> Basic; LCSC (none) -> C20917; Manufacturer Generic -> Alpha & Omega / compatible
- R1: JLCPCB_Type (none) -> Basic; LCSC (none) -> C4190; MPN (none) -> 0603WAF2201T5E; Manufacturer Generic -> UNI-ROYAL
- R2: JLCPCB_Type (none) -> Basic; LCSC (none) -> C22775; MPN (none) -> 0603WAF1000T5E; Manufacturer Generic -> UNI-ROYAL
- R3: JLCPCB_Type (none) -> Basic; LCSC (none) -> C25803; MPN (none) -> 0603WAF1003T5E; Manufacturer Generic -> UNI-ROYAL
- S1: JLCPCB_Type (none) -> Extended; LCSC (none) -> C221841; MPN PCM12-style -> PCM12SMTR; Manufacturer Generic -> Korean Hroparts / compatible
- U1: JLCPCB_Type (none) -> Extended; LCSC (none) -> C5360767
Changed lines of the file:
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@@
 (property "MPN" "DA14531MOD-00F01002" (at 100.33 80.01 0) (effects (font (size 1.27 1.27)) (hide yes)))
 (property "Manufacturer" "Renesas / Dialog" (at 100.33 80.01 0) (effects (font (size 1.27 1.27)) (hide yes)))
+(property "JLCPCB_Type" "Extended" (at 100.33 80.01 0) (effects (font (size 1.27 1.27)) (hide yes)))
+(property "LCSC" "C5360767" (at 100.33 80.01 0) (effects (font (size 1.27 1.27)) (hide yes)))
 (pin "J1")
 (pin "J2")
@@
 (property "MPN" "BH-123A-A1CJ002" (at 35.56 44.45 0) (effects (font (size 1.27 1.27)) (hide yes)))
 (property "Manufacturer" "MYOUNG" (at 35.56 44.45 0) (effects (font (size 1.27 1.27)) (hide yes)))
+(property "JLCPCB_Type" "Extended" (at 35.56 44.45 0) (effects (font (size 1.27 1.27)) (hide yes)))
 (pin "1")
 (pin "2")
@@
 (property "Footprint" "Button_Switch_SMD:SW_SPDT_PCM12" (at 59.69 44.45 0) (effects (font (size 1.27 1.27)) (hide yes)))
 (property "Datasheet" "~" (at 59.69 44.45 0) (effects (font (size 1.27 1.27)) (hide yes)))
-(property "Manufacturer" "Generic" (at 59.69 44.45 0) (effects (font (size 1.27 1.27)) (hide yes)))
-(property "MPN" "PCM12-style" (at 59.69 44.45 0) (effects (font (size 1.27 1.27)) (hide yes)))
+(property "Manufacturer" "Korean Hroparts / compatible" (at 59.69 44.45 0) (effects (font (size 1.27 1.27)) (hide yes)))
+(property "JLCPCB_Type" "Extended" (at 59.69 44.45 0) (effects (font (size 1.27 1.27)) (hide yes)))
+(property "LCSC" "C221841" (at 59.69 44.45 0) (effects (font (size 1.27 1.27)) (hide yes)))
+(property "MPN" "PCM12SMTR" (at 59.69 44.45 0) (effects (font (size 1.27 1.27)) (hide yes)))
 (pin "1")
 (pin "2")
@@
 (property "Footprint" "Capacitor_SMD:C_0805_2012Metric" (at 44.45 74.93 0) (effects (font (size 1.27 1.27)) (hide yes)))
 (property "Datasheet" "~" (at 44.45 74.93 0) (effects (font (size 1.27 1.27)) (hide yes)))
-(property "Manufacturer" "Generic" (at 44.45 74.93 0) (effects (font (size 1.27 1.27)) (hide yes)))
+(property "Manufacturer" "Murata" (at 44.45 74.93 0) (effects (font (size 1.27 1.27)) (hide yes)))
+(property "JLCPCB_Type" "Basic" (at 44.45 74.93 0) (effects (font (size 1.27 1.27)) (hide yes)))
+(property "MPN" "GRM21BR61H106KE43L" (at 44.45 74.93 0) (effects (font (size 1.27 1.27)) (hide yes)))
+(property "LCSC" "C440198" (at 44.45 74.93 0) (effects (font (size 1.27 1.27)) (hide yes)))
 (pin "1")
 (pin "2")
@@
 (property "Footprint" "Capacitor_SMD:C_0603_1608Metric" (at 44.45 82.55 0) (effects (font (size 1.27 1.27)) (hide yes)))
 (property "Datasheet" "~" (at 44.45 82.55 0) (effects (font (size 1.27 1.27)) (hide yes)))
-(property "Manufacturer" "Generic" (at 44.45 82.55 0) (effects (font (size 1.27 1.27)) (hide yes)))
+(property "Manufacturer" "YAGEO" (at 44.45 82.55 0) (effects (font (size 1.27 1.27)) (hide yes)))
+(property "JLCPCB_Type" "Basic" (at 44.45 82.55 0) (effects (font (size 1.27 1.27)) (hide yes)))
+(property "MPN" "CC0603KRX7R9BB104" (at 44.45 82.55 0) (effects (font (size 1.27 1.27)) (hide yes)))
+(property "LCSC" "C14663" (at 44.45 82.55 0) (effects (font (size 1.27 1.27)) (hide yes)))
 (pin "1")
 (pin "2")
@@
 (property "Footprint" "Capacitor_SMD:C_1210_3225Metric" (at 44.45 91.44 0) (effects (font (size 1.27 1.27)) (hide yes)))
 (property "Datasheet" "~" (at 44.45 91.44 0) (effects (font (size 1.27 1.27)) (hide yes)))
-(property "Manufacturer" "Generic" (at 44.45 91.44 0) (effects (font (size 1.27 1.27)) (hide yes)))
+(property "Manufacturer" "Samsung Electro-Mechanics" (at 44.45 91.44 0) (effects (font (size 1.27 1.27)) (hide yes)))
+(property "JLCPCB_Type" "Extended" (at 44.45 91.44 0) (effects (font (size 1.27 1.27)) (hide yes)))
+(property "MPN" "CL32A107MQVNNNE" (at 44.45 91.44 0) (effects (font (size 1.27 1.27)) (hide yes)))
+(property "LCSC" "C49066" (at 44.45 91.44 0) (effects (font (size 1.27 1.27)) (hide yes)))
 (pin "1")
 (pin "2")
@@
 		(property "MPN" "FUET-1365-3V" (at 54.61 119.38 0) (effects (font (size 1.27 1.27)) (hide yes)))
 		(property "Manufacturer" "FUET / Fusheng Electronics" (at 54.61 119.38 0) (effects (font (size 1.27 1.27)) (hide yes)))
+		(property "JLCPCB_Type" "Extended" (at 54.61 119.38 0) (effects (font (size 1.27 1.27)) (hide yes)))
 (pin "1")
 (pin "2")
@@
 (property "Datasheet" "~" (at 85.09 119.38 0) (effects (font (size 1.27 1.27)) (hide yes)))
 (property "MPN" "AO3400A" (at 85.09 119.38 0) (effects (font (size 1.27 1.27)) (hide yes)))
-(property "Manufacturer" "Generic" (at 85.09 119.38 0) (effects (font (size 1.27 1.27)) (hide yes)))
+(property "Manufacturer" "Alpha & Omega / compatible" (at 85.09 119.38 0) (effects (font (size 1.27 1.27)) (hide yes)))
+(property "JLCPCB_Type" "Basic" (at 85.09 119.38 0) (effects (font (size 1.27 1.27)) (hide yes)))
+(property "LCSC" "C20917" (at 85.09 119.38 0) (effects (font (size 1.27 1.27)) (hide yes)))
 (pin "1")
 (pin "2")
@@
 (property "Footprint" "Resistor_SMD:R_0603_1608Metric" (at 69.85 110.49 0) (effects (font (size 1.27 1.27)) (hide yes)))
 (property "Datasheet" "~" (at 69.85 110.49 0) (effects (font (size 1.27 1.27)) (hide yes)))
-(property "Manufacturer" "Generic" (at 69.85 110.49 0) (effects (font (size 1.27 1.27)) (hide yes)))
+(property "Manufacturer" "UNI-ROYAL" (at 69.85 110.49 0) (effects (font (size 1.27 1.27)) (hide yes)))
+(property "JLCPCB_Type" "Basic" (at 69.85 110.49 0) (effects (font (size 1.27 1.27)) (hide yes)))
+(property "MPN" "0603WAF1000T5E" (at 69.85 110.49 0) (effects (font (size 1.27 1.27)) (hide yes)))
+(property "LCSC" "C22775" (at 69.85 110.49 0) (effects (font (size 1.27 1.27)) (hide yes)))
 (pin "1")
 (pin "2")
@@
 (property "Footprint" "Resistor_SMD:R_0603_1608Metric" (at 85.09 132.08 0) (effects (font (size 1.27 1.27)) (hide yes)))
 (property "Datasheet" "~" (at 85.09 132.08 0) (effects (font (size 1.27 1.27)) (hide yes)))
-(property "Manufacturer" "Generic" (at 85.09 132.08 0) (effects (font (size 1.27 1.27)) (hide yes)))
+(property "Manufacturer" "UNI-ROYAL" (at 85.09 132.08 0) (effects (font (size 1.27 1.27)) (hide yes)))
+(property "JLCPCB_Type" "Basic" (at 85.09 132.08 0) (effects (font (size 1.27 1.27)) (hide yes)))
+(property "MPN" "0603WAF1003T5E" (at 85.09 132.08 0) (effects (font (size 1.27 1.27)) (hide yes)))
+(property "LCSC" "C25803" (at 85.09 132.08 0) (effects (font (size 1.27 1.27)) (hide yes)))
 (pin "1")
 (pin "2")
@@
 (property "Footprint" "Diode_SMD:D_SOD-323" (at 69.85 128.27 0) (effects (font (size 1.27 1.27)) (hide yes)))
 (property "Datasheet" "~" (at 69.85 128.27 0) (effects (font (size 1.27 1.27)) (hide yes)))
-(property "MPN" "BAT54WS" (at 69.85 128.27 0) (effects (font (size 1.27 1.27)) (hide yes)))
+(property "MPN" "BAT54WS L9" (at 69.85 128.27 0) (effects (font (size 1.27 1.27)) (hide yes)))
 (property "Manufacturer" "Generic" (at 69.85 128.27 0) (effects (font (size 1.27 1.27)) (hide yes)))
+(property "JLCPCB_Type" "Extended" (at 69.85 128.27 0) (effects (font (size 1.27 1.27)) (hide yes)))
+(property "LCSC" "C22629" (at 69.85 128.27 0) (effects (font (size 1.27 1.27)) (hide yes)))
 (pin "1")
 (pin "2")
@@
 (property "Footprint" "Resistor_SMD:R_0603_1608Metric" (at 129.54 119.38 0) (effects (font (size 1.27 1.27)) (hide yes)))
 (property "Datasheet" "~" (at 129.54 119.38 0) (effects (font (size 1.27 1.27)) (hide yes)))
-(property "Manufacturer" "Generic" (at 129.54 119.38 0) (effects (font (size 1.27 1.27)) (hide yes)))
+(property "Manufacturer" "UNI-ROYAL" (at 129.54 119.38 0) (effects (font (size 1.27 1.27)) (hide yes)))
+(property "JLCPCB_Type" "Basic" (at 129.54 119.38 0) (effects (font (size 1.27 1.27)) (hide yes)))
+(property "MPN" "0603WAF2201T5E" (at 129.54 119.38 0) (effects (font (size 1.27 1.27)) (hide yes)))
+(property "LCSC" "C4190" (at 129.54 119.38 0) (effects (font (size 1.27 1.27)) (hide yes)))
 (pin "1")
 (pin "2")
@@
 (property "Footprint" "LED_SMD:LED_0603_1608Metric" (at 144.78 119.38 0) (effects (font (size 1.27 1.27)) (hide yes)))
 (property "Datasheet" "~" (at 144.78 119.38 0) (effects (font (size 1.27 1.27)) (hide yes)))
-(property "Manufacturer" "Generic" (at 144.78 119.38 0) (effects (font (size 1.27 1.27)) (hide yes)))
-(pin "1")
-(pin "2")
+(property "Manufacturer" "KENTO" (at 144.78 119.38 0) (effects (font (size 1.27 1.27)) (hide yes)))
+(property "JLCPCB_Type" "Basic" (at 144.78 119.38 0) (effects (font (size 1.27 1.27)) (hide yes)))
+(property "MPN" "KT-0603R" (at 144.78 119.38 0) (effects (font (size 1.27 1.27)) (hide yes)))
+(property "LCSC" "C2286" (at 144.78 119.38 0) (effects (font (size 1.27 1.27)) (hide yes)))
+(pin "1")
+(pin "2")

Commit message: Checkpoint before Buzzer CR2450 redesign
Parts:
- BT1: value BH-123A-A1CJ002 CR123A holder candidate -> Keystone 3008 CR2450 holder; footprint SafeGuardBuzzer_Local:BatteryHolder_CR123A_MYOUNG_BH-123A-A1CJ002_C5290177_THT -> SafeGuardBuzzer_Local:BatteryHolder_Keystone_3008_1x2450; symbol SafeGuardBuzzer_Local:Battery_CR123A_1Cell -> SafeGuardBuzzer_Local:Battery_CR2450_1Cell; LCSC C5290177 -> (none); MPN BH-123A-A1CJ002 -> 3008; Manufacturer MYOUNG -> Keystone
Changed lines of the file:
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@@
 (no_connect (at 115.57 87.63))
 (no_connect (at 115.57 90.17))
-(symbol (lib_id "SafeGuardBuzzer_Local:Battery_CR123A_1Cell") (at 35.56 44.45 0) (unit 1) (exclude_from_sim no) (in_bom yes) (on_board yes) (dnp no)
+(symbol (lib_id "SafeGuardBuzzer_Local:Battery_CR2450_1Cell") (at 35.56 44.45 0) (unit 1) (exclude_from_sim no) (in_bom yes) (on_board yes) (dnp no)
 (property "Reference" "BT1" (at 35.56 39.37 0) (effects (font (size 1.27 1.27))))
-(property "Value" "BH-123A-A1CJ002 CR123A holder candidate" (at 35.56 49.53 0) (effects (font (size 1.27 1.27))))
-		(property "Footprint" "SafeGuardBuzzer_Local:BatteryHolder_CR123A_MYOUNG_BH-123A-A1CJ002_C5290177_THT" (at 35.56 44.45 0) (effects (font (size 1.27 1.27)) (hide yes)))
-(property "Datasheet" "~" (at 35.56 44.45 0) (effects (font (size 1.27 1.27)) (hide yes)))
-(property "LCSC" "C5290177" (at 35.56 44.45 0) (effects (font (size 1.27 1.27)) (hide yes)))
-(property "MPN" "BH-123A-A1CJ002" (at 35.56 44.45 0) (effects (font (size 1.27 1.27)) (hide yes)))
-(property "Manufacturer" "MYOUNG" (at 35.56 44.45 0) (effects (font (size 1.27 1.27)) (hide yes)))
+(property "Value" "Keystone 3008 CR2450 holder" (at 35.56 49.53 0) (effects (font (size 1.27 1.27))))
+		(property "Footprint" "SafeGuardBuzzer_Local:BatteryHolder_Keystone_3008_1x2450" (at 35.56 44.45 0) (effects (font (size 1.27 1.27)) (hide yes)))
+		(property "Datasheet" "http://www.keyelco.com/product-pdf.cfm?p=786" (at 35.56 44.45 0) (effects (font (size 1.27 1.27)) (hide yes)))
+(property "LCSC" "" (at 35.56 44.45 0) (effects (font (size 1.27 1.27)) (hide yes)))
+(property "MPN" "3008" (at 35.56 44.45 0) (effects (font (size 1.27 1.27)) (hide yes)))
+		(property "Manufacturer" "Keystone" (at 35.56 44.45 0) (effects (font (size 1.27 1.27)) (hide yes)))
 (property "JLCPCB_Type" "Extended" (at 35.56 44.45 0) (effects (font (size 1.27 1.27)) (hide yes)))
 (pin "1")

Commit message: Redesign Buzzer v1 for CR2450 battery
Parts:
- BT1: value Keystone 3008 CR2450 holder -> MYOUNG MY-2450-03 CR2450 holder; footprint SafeGuardBuzzer_Local:BatteryHolder_Keystone_3008_1x2450 -> SafeGuardBuzzer_Local:BatteryHolder_MYOUNG_MY-2450-03_C2988622_CR2450; LCSC (none) -> C2988622; MPN 3008 -> MY-2450-03; Manufacturer Keystone -> MYOUNG
Changed lines of the file:
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@@
 (symbol (lib_id "SafeGuardBuzzer_Local:Battery_CR2450_1Cell") (at 35.56 44.45 0) (unit 1) (exclude_from_sim no) (in_bom yes) (on_board yes) (dnp no)
 (property "Reference" "BT1" (at 35.56 39.37 0) (effects (font (size 1.27 1.27))))
-(property "Value" "Keystone 3008 CR2450 holder" (at 35.56 49.53 0) (effects (font (size 1.27 1.27))))
-		(property "Footprint" "SafeGuardBuzzer_Local:BatteryHolder_Keystone_3008_1x2450" (at 35.56 44.45 0) (effects (font (size 1.27 1.27)) (hide yes)))
-		(property "Datasheet" "http://www.keyelco.com/product-pdf.cfm?p=786" (at 35.56 44.45 0) (effects (font (size 1.27 1.27)) (hide yes)))
-(property "LCSC" "" (at 35.56 44.45 0) (effects (font (size 1.27 1.27)) (hide yes)))
-(property "MPN" "3008" (at 35.56 44.45 0) (effects (font (size 1.27 1.27)) (hide yes)))
-		(property "Manufacturer" "Keystone" (at 35.56 44.45 0) (effects (font (size 1.27 1.27)) (hide yes)))
+(property "Value" "MYOUNG MY-2450-03 CR2450 holder" (at 35.56 49.53 0) (effects (font (size 1.27 1.27))))
+		(property "Footprint" "SafeGuardBuzzer_Local:BatteryHolder_MYOUNG_MY-2450-03_C2988622_CR2450" (at 35.56 44.45 0) (effects (font (size 1.27 1.27)) (hide yes)))
+		(property "Datasheet" "https://wmsc.lcsc.com/wmsc/upload/file/pdf/v2/lcsc/2204021730_MYOUNG-MY-2450-03_C2988622.pdf" (at 35.56 44.45 0) (effects (font (size 1.27 1.27)) (hide yes)))
+(property "LCSC" "C2988622" (at 35.56 44.45 0) (effects (font (size 1.27 1.27)) (hide yes)))
+(property "MPN" "MY-2450-03" (at 35.56 44.45 0) (effects (font (size 1.27 1.27)) (hide yes)))
+		(property "Manufacturer" "MYOUNG" (at 35.56 44.45 0) (effects (font (size 1.27 1.27)) (hide yes)))
 (property "JLCPCB_Type" "Extended" (at 35.56 44.45 0) (effects (font (size 1.27 1.27)) (hide yes)))
 (pin "1")

Commit message: PCB contains copper zones near C3; fixed it
Parts:
- C3: footprint Capacitor_SMD:C_1210_3225Metric -> SafeGuardBuzzer_Local:C_1210_3225_Samsung_CL32A107MQVNNNE_C49066
Changed lines of the file:
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@@
 (property "Reference" "C3" (at 44.45 86.36 0) (effects (font (size 1.27 1.27))))
 (property "Value" "100uF 6.3V bulk" (at 44.45 96.52 0) (effects (font (size 1.27 1.27))))
-(property "Footprint" "Capacitor_SMD:C_1210_3225Metric" (at 44.45 91.44 0) (effects (font (size 1.27 1.27)) (hide yes)))
+(property "Footprint" "SafeGuardBuzzer_Local:C_1210_3225_Samsung_CL32A107MQVNNNE_C49066" (at 44.45 91.44 0) (effects (font (size 1.27 1.27)) (hide yes)))
 (property "Datasheet" "~" (at 44.45 91.44 0) (effects (font (size 1.27 1.27)) (hide yes)))
 (property "Manufacturer" "Samsung Electro-Mechanics" (at 44.45 91.44 0) (effects (font (size 1.27 1.27)) (hide yes)))
